Commit message: work in progress....

File: new_React/ONS/public/ur5.urdf (robot description, URDF)
Before this commit: robot ur5, 7 links, 6 joints
Links:
- link base_link: mass None -> 4
- link forearm_link: mass None -> 2.275
- link shoulder_link: mass None -> 3.7
- link upper_arm_link: mass None -> 8.393
- link wrist_1_link: mass None -> 1.219
- link wrist_2_link: mass None -> 1.219
- link wrist_3_link: mass None -> 0.1879
Joints:
- joint elbow_joint: limit lower=-6.283185 upper=6.283185 effort=150 velocity=3.14159 -> lower=-6.283185 upper=6.283185 effort=150 velocity=3.15
- joint shoulder_lift_joint: limit lower=-6.283185 upper=6.283185 effort=150 velocity=3.14159 -> lower=-6.283185 upper=6.283185 effort=150 velocity=3.15
- joint shoulder_pan_joint: limit lower=-6.283185 upper=6.283185 effort=150 velocity=3.14159 -> lower=-6.283185 upper=6.283185 effort=150 velocity=3.15
- joint wrist_1_joint: limit lower=-6.283185 upper=6.283185 effort=28 velocity=3.14159 -> lower=-6.283185 upper=6.283185 effort=28 velocity=3.2
- joint wrist_2_joint: limit lower=-6.283185 upper=6.283185 effort=28 velocity=3.14159 -> lower=-6.283185 upper=6.283185 effort=28 velocity=3.2
- joint wrist_3_joint: limit lower=-6.283185 upper=6.283185 effort=28 velocity=3.14159 -> lower=-6.283185 upper=6.283185 effort=28 velocity=3.2
